File: TX5823/TX5823.sch (KiCad schematic (older format))
At the start: 0 parts

Commit message: Bauteile angelegt
Parts:
- added IC?: ATMEGA328P-A, TQFP32, symbol ATMEGA328P-A
- added IC?: ATTINY13A-SS, SO8, symbol ATTINY13A-SS
- added R?: 10k, symbol R
- added U?: TPS54531, symbol TPS54531
- added U?: TX5823, symbol TX5823
- added U?: MAX7456_DS, symbol MAX7456_DS
- added U?: TPS7A7200RGT, symbol TPS7A7200RGT
- added U?: LM25118, symbol LM25118
Connections:
- new net: IC?.5 (PB0(MOSI/AIN0/OC0A/PCINT0)), U?.6 (CH1/SPIDATA)
- new net: IC?.3 (PB4(ADC2/PCINT4)), R?.2, U?.7 (CH2/SPILE)
- new net: IC?.7 (PB2(SCK/ADC1/T0/PCINT2)), U?.8 (CH3/SPICLK)
- new net +3.3V: R?.1
Other:
- note added: "5V_Stepdown"
- note added: "TODO\nBOOST\nEP anpassen\n"
Changed lines of the file:
@@
 LIBS:contrib
 LIBS:valves
+LIBS:toni
+LIBS:TX5823-cache
 EELAYER 25 0
 EELAYER END
@@
 Comment4 ""
 $EndDescr
+$Comp
+L TPS54531 U?
+U 1 1 5513E458
+P 3450 2150
+F 0 "U?" H 3850 1300 60  0000 C CNN
+F 1 "TPS54531" H 3450 2950 60  0000 C CNN
+F 2 "" H 3500 2150 60  0000 C CNN
+F 3 "" H 3500 2150 60  0000 C CNN
+	1    3450 2150
+	1    0    0    -1
+$EndComp
+Text Notes 3200 1250 0    60   ~ 0
+5V_Stepdown
+$Comp
+L TX5823 U?
+U 1 1 5513E991
+P 9350 1700
+F 0 "U?" H 9900 750 60  0000 C CNN
+F 1 "TX5823" H 9500 1400 60  0000 C CNN
+F 2 "" H 9200 1650 60  0000 C CNN
+F 3 "" H 9200 1650 60  0000 C CNN
+	1    9350 1700
+	1    0    0    -1
+$EndComp
+$Comp
+L MAX7456_DS U?
+U 1 1 551495BC
+P 5950 5150
+F 0 "U?" H 6500 4550 60  0000 C CNN
+F 1 "MAX7456_DS" H 6100 6000 60  0000 C CNN
+F 2 "" H 5950 5150 60  0000 C CNN
+F 3 "" H 5950 5150 60  0000 C CNN
+	1    5950 5150
+	1    0    0    -1
+$EndComp
+$Comp
+L ATMEGA328P-A IC?
+U 1 1 5514960B
+P 3250 5500
+F 0 "IC?" H 2500 6750 40  0000 L BNN
+F 1 "ATMEGA328P-A" H 3650 4100 40  0000 L BNN
+F 2 "TQFP32" H 3250 5500 30  0000 C CIN
+F 3 "" H 3250 5500 60  0000 C CNN
+	1    3250 5500
+	1    0    0    -1
+$EndComp
+$Comp
+L ATTINY13A-SS IC?
+U 1 1 551496E8
+P 6950 2100
+F 0 "IC?" H 6150 2500 40  0000 C CNN
+F 1 "ATTINY13A-SS" H 7600 1700 40  0000 C CNN
+F 2 "SO8" H 7550 2100 35  0000 C CIN
+F 3 "" H 6150 2450 60  0000 C CNN
+	1    6950 2100
+	-1   0    0    -1
+$EndComp
+Wire Wire Line
+	7950 1850 8600 1850
+Wire Wire Line
+	7950 2050 8450 2050
+Wire Wire Line
+	8450 2050 8450 2150
+Wire Wire Line
+	8450 2150 8600 2150
+Wire Wire Line
+	8350 2000 8600 2000
+Wire Wire Line
+	8350 1250 8350 2250
+Wire Wire Line
+	8350 2250 7950 2250
+$Comp
+L R R?
+U 1 1 55149D57
+P 8350 1000
+F 0 "R?" V 8430 1000 40  0000 C CNN
+F 1 "10k" V 8357 1001 40  0000 C CNN
+F 2 "" V 8280 1000 30  0000 C CNN
+F 3 "" H 8350 1000 30  0000 C CNN
+	1    8350 1000
+	1    0    0    -1
+$EndComp
+Connection ~ 8350 2000
+$Comp
+L +3,3V #PWR?
+U 1 1 55149E19
+P 8350 750
+F 0 "#PWR?" H 8350 710 30  0001 C CNN
+F 1 "+3,3V" H 8350 860 30  0000 C CNN
+F 2 "" H 8350 750 60  0000 C CNN
+F 3 "" H 8350 750 60  0000 C CNN
+	1    8350 750
+	1    0    0    -1
+$EndComp
+Text Notes 800  1700 0    197  ~ 0
+TODO\nBOOST\nEP anpassen\n
+$Comp
+L TPS7A7200RGT U?
+U 1 1 5514B0D0
+P 4950 1950
+F 0 "U?" H 5400 1500 60  0000 C CNN
+F 1 "TPS7A7200RGT" H 4950 2600 60  0000 C CNN
+F 2 "" H 4950 1950 60  0000 C CNN
+F 3 "" H 4950 1950 60  0000 C CNN
+	1    4950 1950
+	1    0    0    -1
+$EndComp
+$Comp
+L LM25118 U?
+U 1 1 5514C262
+P 9500 4950
+F 0 "U?" H 9800 4100 60  0000 C CNN
+F 1 "LM25118" H 9500 5750 60  0000 C CNN
+F 2 "" H 9300 4950 60  0000 C CNN
+F 3 "" H 9300 4950 60  0000 C CNN
+	1    9500 4950
+	1    0    0    -1
+$EndComp
 $EndSCHEMATC
