File: TX5823/TX5823.sch (KiCad schematic (older format))
At the start: 95 parts

Commit message: Schaltplan bereit für review
Parts:
- added P?: Akku_in, symbol CONN_01X02
- P?: value CONN_02X03 -> ISP
- RP?: value R_PACK4 -> 1k
Connections:
- net GND: now also P?.1 (P1)
- net Akku+: now reaches C?.1, C?.1, U?.2 (VIN)
- net Akku+: now also C?.1, C?.1, Q?.D, R?.1, R?.1, U?.1 (VIN), P?.2 (P2)
Other:
- note added: "Buck\nVin 8V-28V\n5V Stepdown\n5A out"
- note added: "TODO:\nSMA Buchse"
- note added: "laut Beispiel im Datenblatt\nRcomp 37.4k\nCcomp= 2200pF\nCcomp2=22pF\nl=4,7 uH\nAchtung, teilweise Teilenummern aus der 5A webbranch\nKalkulation übernommen\n\n"
- note removed: "Vin 8V-28V\n5V Stepdown\n5A out"
- note removed: "laut Beispiel im Datenblatt\nRcomp 37.4k\nCcomp= 2200pF\nCcomp2=22pF\nl=4,7 uH\nAchtung, Teilenummern aus der 5A webbranche\nKalkulation übernommen\n\n"
- moved on the sheet: P?, R?, SW?, U?
Changed lines of the file:
@@
 	1    0    0    -1
 $EndComp
-Text Notes 950  7100 0    197  ~ 0
-Vin 8V-28V\n5V Stepdown\n5A out
+Text Notes 950  7300 0    197  ~ 0
+Buck\nVin 8V-28V\n5V Stepdown\n5A out
 $Comp
 L TX5823 U?
@@
 P 14950 4900
 F 0 "RP?" H 14950 5350 40  0000 C CNN
-F 1 "R_PACK4" H 14950 4850 40  0000 C CNN
+F 1 "1k" H 14950 4850 40  0000 C CNN
 F 2 "" H 14950 4900 60  0000 C CNN
 F 3 "" H 14950 4900 60  0000 C CNN
@@
 P 14100 4900
 F 0 "P?" H 14100 5100 50  0000 C CNN
-F 1 "CONN_02X03" H 14100 4700 50  0000 C CNN
+F 1 "ISP" H 14100 4700 50  0000 C CNN
 F 2 "" H 14100 3700 60  0000 C CNN
 F 3 "" H 14100 3700 60  0000 C CNN
@@
 $EndComp
 Text Notes 3450 7000 0    60   ~ 0
-laut Beispiel im Datenblatt\nRcomp 37.4k\nCcomp= 2200pF\nCcomp2=22pF\nl=4,7 uH\nAchtung, Teilenummern aus der 5A webbranche\nKalkulation übernommen\n\n
+laut Beispiel im Datenblatt\nRcomp 37.4k\nCcomp= 2200pF\nCcomp2=22pF\nl=4,7 uH\nAchtung, teilweise Teilenummern aus der 5A webbranch\nKalkulation übernommen\n\n
 $Comp
 L C C?
@@
 L CONN_01X05 P?
 U 1 1 5517FDD8
-P 15050 8900
-F 0 "P?" H 15050 9200 50  0000 C CNN
-F 1 "Mavlink" V 15150 8900 50  0000 C CNN
-F 2 "" H 15050 8900 60  0000 C CNN
-F 3 "" H 15050 8900 60  0000 C CNN
-	1    15050 8900
+P 15700 8900
+F 0 "P?" H 15700 9200 50  0000 C CNN
+F 1 "Mavlink" V 15800 8900 50  0000 C CNN
+F 2 "" H 15700 8900 60  0000 C CNN
+F 3 "" H 15700 8900 60  0000 C CNN
+	1    15700 8900
 	1    0    0    -1
 $EndComp
@@
 Text Label 9350 9800 1    60   ~ 0
 IR_LED+
-Text Label 14850 8700 2    60   ~ 0
+Text Label 15500 8700 2    60   ~ 0
 DTR
-Text Label 14350 8800 2    60   ~ 0
+Text Label 15000 8800 2    60   ~ 0
 TXO
-Text Label 13100 8900 2    60   ~ 0
+Text Label 13750 8900 2    60   ~ 0
 RXI
 $Comp
 L +5V #PWR?
 U 1 1 55194093
-P 14850 9000
-F 0 "#PWR?" H 14850 9090 20  0001 C CNN
-F 1 "+5V" H 14850 9090 30  0000 C CNN
-F 2 "" H 14850 9000 60  0000 C CNN
-F 3 "" H 14850 9000 60  0000 C CNN
-	1    14850 9000
+P 15500 9000
+F 0 "#PWR?" H 15500 9090 20  0001 C CNN
+F 1 "+5V" H 15500 9090 30  0000 C CNN
+F 2 "" H 15500 9000 60  0000 C CNN
+F 3 "" H 15500 9000 60  0000 C CNN
+	1    15500 9000
 	0    -1   -1   0
 $EndComp
@@
 L R R?
 U 1 1 551949B3
-P 14600 8800
-F 0 "R?" V 14680 8800 40  0000 C CNN
-F 1 "100R" V 14607 8801 40  0000 C CNN
-F 2 "" V 14530 8800 30  0000 C CNN
-F 3 "" V 14680 8800 30  0000 C CNN
-	1    14600 8800
+P 15250 8800
+F 0 "R?" V 15330 8800 40  0000 C CNN
+F 1 "100R" V 15257 8801 40  0000 C CNN
+F 2 "" V 15180 8800 30  0000 C CNN
+F 3 "" V 15330 8800 30  0000 C CNN
+	1    15250 8800
 	0    1    1    0
 $EndComp
@@
 L OPTO-TRANSISTOR4 U?
 U 1 1 5519658E
-P 13700 9050
-F 0 "U?" H 13900 9300 60  0000 C CNN
-F 1 "OPTO-TRANSISTOR4" H 13700 8800 60  0000 C CNN
-F 2 "" H 13700 9050 60  0000 C CNN
-F 3 "" H 13700 9050 60  0000 C CNN
-	1    13700 9050
+P 14350 9050
+F 0 "U?" H 14550 9300 60  0000 C CNN
+F 1 "OPTO-TRANSISTOR4" H 14350 8800 60  0000 C CNN
+F 2 "" H 14350 9050 60  0000 C CNN
+F 3 "" H 14350 9050 60  0000 C CNN
+	1    14350 9050
 	-1   0    0    -1
 $EndComp
@@
 L R R?
 U 1 1 55197380
-P 14600 8900
-F 0 "R?" V 14680 8900 40  0000 C CNN
-F 1 "300R" V 14607 8901 40  0000 C CNN
-F 2 "" V 14530 8900 30  0000 C CNN
-F 3 "" V 14680 8900 30  0000 C CNN
-	1    14600 8900
+P 15250 8900
+F 0 "R?" V 15330 8900 40  0000 C CNN
+F 1 "300R" V 15257 8901 40  0000 C CNN
+F 2 "" V 15180 8900 30  0000 C CNN
+F 3 "" V 15330 8900 30  0000 C CNN
+	1    15250 8900
 	0    1    1    0
 $EndComp
@@
 L +5V #PWR?
 U 1 1 55198D20
-P 13100 8400
-F 0 "#PWR?" H 13100 8490 20  0001 C CNN
-F 1 "+5V" H 13100 8490 30  0000 C CNN
-F 2 "" H 13100 8400 60  0000 C CNN
-F 3 "" H 13100 8400 60  0000 C CNN
-	1    13100 8400
+P 13750 8400
+F 0 "#PWR?" H 13750 8490 20  0001 C CNN
+F 1 "+5V" H 13750 8490 30  0000 C CNN
+F 2 "" H 13750 8400 60  0000 C CNN
+F 3 "" H 13750 8400 60  0000 C CNN
+	1    13750 8400
 	1    0    0    -1
 $EndComp
@@
 L R R?
 U 1 1 5519918F
-P 13100 8650
-F 0 "R?" V 13180 8650 40  0000 C CNN
-F 1 "open" V 13107 8651 40  0000 C CNN
-F 2 "Resistors_SMD:R_0603" V 13030 8650 30  0001 C CNN
-F 3 "" V 13180 8650 30  0000 C CNN
-	1    13100 8650
+P 13750 8650
+F 0 "R?" V 13830 8650 40  0000 C CNN
+F 1 "open" V 13757 8651 40  0000 C CNN
+F 2 "Resistors_SMD:R_0603" V 13680 8650 30  0001 C CNN
+F 3 "" V 13830 8650 30  0000 C CNN
+	1    13750 8650
 	1    0    0    -1
 $EndComp
@@
 L GND #PWR?
 U 1 1 55199759
-P 13100 9550
-F 0 "#PWR?" H 13100 9550 30  0001 C CNN
-F 1 "GND" H 13100 9480 30  0001 C CNN
-F 2 "" H 13100 9550 60  0000 C CNN
-F 3 "" H 13100 9550 60  0000 C CNN
-	1    13100 9550
-	1    0    0    -1
-$EndComp
-Wire Wire Line
-	14350 9200 14450 9200
-Wire Wire Line
-	14450 9200 14450 9100
-Wire Wire Line
-	14450 9100 14850 9100
-Connection ~ 13100 9500
-Wire Wire Line
-	13100 9200 13100 9550
-Wire Wire Line
-	13100 9500 13350 9500
+P 13750 9550
+F 0 "#PWR?" H 13750 9550 30  0001 C CNN
+F 1 "GND" H 13750 9480 30  0001 C CNN
+F 2 "" H 13750 9550 60  0000 C CNN
+F 3 "" H 13750 9550 60  0000 C CNN
+	1    13750 9550
+	1    0    0    -1
+$EndComp
+Wire Wire Line
+	15000 9200 15100 9200
+Wire Wire Line
+	15100 9200 15100 9100
+Wire Wire Line
+	15100 9100 15500 9100
+Connection ~ 13750 9500
+Wire Wire Line
+	13750 9200 13750 9550
+Wire Wire Line
+	13750 9500 14000 9500
 $Comp
 L SW_PUSH SW?
 U 1 1 5519BDF1
-P 13650 9500
-F 0 "SW?" H 13800 9610 50  0000 C CNN
-F 1 "SW_PUSH" H 13650 9420 50  0000 C CNN
-F 2 "" H 13650 9500 60  0000 C CNN
-F 3 "" H 13650 9500 60  0000 C CNN
-	1    13650 9500
-	1    0    0    -1
-$EndComp
-Wire Wire Line
-	14350 9500 14350 9200
-Wire Wire Line
-	13950 9500 14350 9500
+P 14300 9500
+F 0 "SW?" H 14450 9610 50  0000 C CNN
+F 1 "SW_PUSH" H 14300 9420 50  0000 C CNN
+F 2 "" H 14300 9500 60  0000 C CNN
+F 3 "" H 14300 9500 60  0000 C CNN
+	1    14300 9500
+	1    0    0    -1
+$EndComp
+Wire Wire Line
+	15000 9500 15000 9200
+Wire Wire Line
+	14600 9500 15000 9500
+Text Label 1200 2300 2    60   ~ 0
+Akku+
+Text Label 1600 8000 2    60   ~ 0
+Akku+
+Text Label 12350 9100 2    60   ~ 0
+Akku+
+$Comp
+L CONN_01X02 P?
+U 1 1 551A56AF
+P 12600 9050
+F 0 "P?" H 12600 9200 50  0000 C CNN
+F 1 "Akku_in" V 12700 9050 50  0000 C CNN
+F 2 "" H 12600 9050 60  0000 C CNN
+F 3 "" H 12600 9050 60  0000 C CNN
+	1    12600 9050
+	1    0    0    -1
+$EndComp
+$Comp
+L GND #PWR?
+U 1 1 551A5702
+P 12400 9000
+F 0 "#PWR?" H 12400 9000 30  0001 C CNN
+F 1 "GND" H 12400 8930 30  0001 C CNN
+F 2 "" H 12400 9000 60  0000 C CNN
+F 3 "" H 12400 9000 60  0000 C CNN
+	1    12400 9000
+	0    1    1    0
+$EndComp
+Wire Wire Line
+	12350 9100 12400 9100
+Wire Notes Line
+	13050 8100 13050 9900
+Text Notes 1200 -1100 0    197  ~ 0
+TODO:\nSMA Buchse
 $EndSCHEMATC

Commit message: ERC errors weitestgehend korrigiert
Parts:
- gave numbers to parts that had none: 96
Connections:
- net SSOD-IN is gone; now on net SSOSD-IN: U7.8 (~CS)
- net +5V: now also C21.1
- no-connect marks 25 -> 28

Commit message: an Schaltplan weitergearbeitet footprints hinzugefügt
Parts:
- added C38: 1uF/50V, Capacitors_SMD:C_1206, symbol C
- added R31: 300R, Capacitors_SMD:C_0805, symbol R
- C10, C15, C2, C4, C7, C9, R29, R30: footprint (none) -> Capacitors_SMD:C_0805
- C12, C13: footprint (none) -> Capacitors_SMD:C_0402
- C18: footprint (none) -> Capacitors_SMD:c_elec_8x10; Teilenummer 16SVP180M -> 20SVPF180M
- C35, C36: footprint (none) -> Capacitors_Tantalum_SMD:TantalC_SizeB_EIA-3528_Reflow
- C37: value 100nF -> 100nF/NP0; footprint (none) -> Capacitors_SMD:C_1206; Teilenummer (none) -> C3216C0G1H104J160AA
- C6: footprint (none) -> Capacitors_SMD:C_1206
- D2, D3, D4, D5: footprint (none) -> Diodes_SMD:Diode-SMC_Standard
- D6: footprint (none) -> LEDs:LED-0603
- IC1: footprint TQFP32 -> Housings_QFP:TQFP-32_7x7mm_Pitch0.8mm
- IC2: footprint SO8 -> SMD_Packages:SOIC-8-N
- P1: footprint (none) -> Socket_Strips:Socket_Strip_Angled_1x02
- P2: footprint (none) -> toni:micro_match3x2
- P3: footprint (none) -> Connectors_Molex:Connector_Molex_PicoBlade_53261-0571
- R1, R2, R3, R4, R5, R7, R8: footprint (none) -> Resistors_SMD:R_0402
- R13, R24, R27, R28: footprint (none) -> Resistors_SMD:R_0603
- R18, R22, R23: footprint (none) -> Resistors_SMD:R_0805
- R9: footprint (none) -> Resistors_SMD:R_1206
- RP1: footprint (none) -> Resistors_SMD:R_Array_Concave_4x0603
- U3: footprint (none) -> Housings_DFN_QFN:QFN-16-1EP_3x3mm_Pitch0.5mm
- U5, U8: footprint (none) -> toni:SO-4
- Y1: footprint (none) -> toni:CerOsc_3,2x1,3
Connections:
- net +12V: now also C38.1
- net GND: now also C38.2
- net PWM_in: now also R31.1; no longer U5.4 (C)
- net at U7.25 (SAG): now also C36.1; no longer C36.2
- net at U7.26 (VOUT): now also C35.1; no longer C35.2
- new net: C35.2, C36.2, R29.2
- new net: R31.2, U5.4 (C)
Other:
- note added: "75Ohm Videosignal routen:\n\nLeitungsbreite 171,25 µm, daneben massefläche mit einem Abstand von 200 µm zur Leitung. \ndarunter Massefläche mit einem Abstand von z=220 µm\nergibt dann 75 R bei FR4"
- note added: "TODO:\nSMA Buchse\nEingangsfilterung (spule und diode)"
- note removed: "TODO:\nSMA Buchse"

Commit message: weitere Footprints zugeordnet grobe Anordnung der Bauteiele im Layout
Parts:
- U1: footprint (none) -> toni:TSSOP-20_4.4x6.5mm_Pitch0.65mm_EP
- U2: footprint (none) -> toni:SO8_EP
- U3: footprint Housings_DFN_QFN:QFN-16-1EP_3x3mm_Pitch0.5mm -> toni:QFN-16-1EP_3x3mm_Pitch0.5mm
- U6: footprint (none) -> toni:TX5823
Changed lines of the file:
@@
 F 0 "U2" H 3900 7750 60  0000 C CNN
 F 1 "TPS54531" H 3500 9400 60  0000 C CNN
-F 2 "" H 3550 8600 60  0001 C CNN
+F 2 "toni:SO8_EP" H 3550 8600 60  0001 C CNN
 F 3 "" H 3550 8600 60  0000 C CNN
 	1    3500 8600
@@
 F 0 "U6" H 14100 900 60  0000 C CNN
 F 1 "TX5823" H 13700 1550 60  0000 C CNN
-F 2 "" H 13400 1800 60  0001 C CNN
+F 2 "toni:TX5823" H 13400 1800 60  0001 C CNN
 F 3 "" H 13400 1800 60  0000 C CNN
 	1    13550 1850
@@
 F 0 "U3" H 9300 1150 60  0000 C CNN
 F 1 "TPS7A7200RGT" H 8850 2250 60  0000 C CNN
-F 2 "Housings_DFN_QFN:QFN-16-1EP_3x3mm_Pitch0.5mm" H 8850 1600 60  0001 C CNN
+F 2 "toni:QFN-16-1EP_3x3mm_Pitch0.5mm" H 8850 1600 60  0001 C CNN
 F 3 "" H 8850 1600 60  0000 C CNN
 	1    8850 1600
@@
 F 0 "U1" H 3800 2800 60  0000 C CNN
 F 1 "LM25118" H 3500 4450 60  0000 C CNN
-F 2 "" H 3300 3650 60  0001 C CNN
+F 2 "toni:TSSOP-20_4.4x6.5mm_Pitch0.65mm_EP" H 3300 3650 60  0001 C CNN
 F 3 "" H 3300 3650 60  0000 C CNN
 	1    3500 3650
