File: TX5823/TX5823.sch (KiCad schematic (older format))
At the start: 98 parts, among them IC1 ATMEGA328P-A, IC2 ATTINY13A-SS, P1 Akku_in, P2 ISP, P3 Mavlink, Q1 MOS_N, Q2 MOS_N, Q3 MOSFET_N, SW1 SW_PUSH, SW2 SW_PUSH, U1 LM25118, U2 TPS54531, U3 TPS7A7200RGT, U4 CONN_03X08, U5 OPTO-TRANSISTOR4, U6 TX5823, U7 MAX7456_DS, U8 OPTO-TRANSISTOR4, X1 27MHz, Y1 16MHz

Commit message: sma buchse hinzugefügt
Parts:
- added SMA_E1: SMA_EDGE, symbol SMA_EDGE
- U7: footprint (none) -> toni:TSSOP-20_4.4x6.5mm_Pitch0.65mm_EP
Connections:
- net GND: now also U6.11 (GND_ANTENNA), SMA_E1.0 (GND), SMA_E1.2 (GND)
- net at U6.10 (ANT): now also SMA_E1.1 (SIGNAL)
Changed lines of the file:
@@
 EESchema Schematic File Version 2
+LIBS:SMA_EDGE
 LIBS:power
 LIBS:device
@@
 LIBS:contrib
 LIBS:valves
+LIBS:Resonator_3pins
+LIBS:rx5808
+LIBS:tps62160
+LIBS:Rafi
 LIBS:toni
-LIBS:TX5823-cache
+LIBS:rx5808_4button-cache
 EELAYER 25 0
 EELAYER END
@@
 F 0 "U7" H 14400 6600 60  0000 C CNN
 F 1 "MAX7456_DS" H 14000 8050 60  0000 C CNN
-F 2 "" H 13850 7200 60  0001 C CNN
+F 2 "toni:TSSOP-20_4.4x6.5mm_Pitch0.65mm_EP" H 13850 7200 60  0001 C CNN
 F 3 "" H 13850 7200 60  0000 C CNN
 	1    13850 7200
@@
 Text Notes 11300 4600 0    60   ~ 0
 75Ohm Videosignal routen:\n\nLeitungsbreite 171,25 µm, daneben massefläche mit einem Abstand von 200 µm zur Leitung. \ndarunter Massefläche mit einem Abstand von z=220 µm\nergibt dann 75 R bei FR4
+$Comp
+L SMA_EDGE SMA_E1
+U 1 1 5518495B
+P 15050 1550
+F 0 "SMA_E1" H 15200 1850 60  0000 C CNN
+F 1 "SMA_EDGE" H 15200 1750 60  0000 C CNN
+F 2 "" H 15050 1550 60  0000 C CNN
+F 3 "" H 15050 1550 60  0000 C CNN
+	1    15050 1550
+	1    0    0    -1
+$EndComp
+Wire Wire Line
+	14250 1550 14700 1550
+$Comp
+L GND #PWR0100
+U 1 1 55184ED5
+P 14700 1650
+F 0 "#PWR0100" H 14700 1650 30  0001 C CNN
+F 1 "GND" H 14700 1580 30  0001 C CNN
+F 2 "" H 14700 1650 60  0000 C CNN
+F 3 "" H 14700 1650 60  0000 C CNN
+	1    14700 1650
+	0    1    1    0
+$EndComp
+$Comp
+L GND #PWR0101
+U 1 1 55184F4A
+P 14700 1450
+F 0 "#PWR0101" H 14700 1450 30  0001 C CNN
+F 1 "GND" H 14700 1380 30  0001 C CNN
+F 2 "" H 14700 1450 60  0000 C CNN
+F 3 "" H 14700 1450 60  0000 C CNN
+	1    14700 1450
+	0    1    1    0
+$EndComp
+$Comp
+L GND #PWR0102
+U 1 1 551851AF
+P 14250 1750
+F 0 "#PWR0102" H 14250 1750 30  0001 C CNN
+F 1 "GND" H 14250 1680 30  0001 C CNN
+F 2 "" H 14250 1750 60  0000 C CNN
+F 3 "" H 14250 1750 60  0000 C CNN
+	1    14250 1750
+	0    -1   -1   0
+$EndComp
 $EndSCHEMATC

Commit message: Bauteile grob angeordnet
Parts:
- L1: footprint (none) -> Choke_SMD:Choke_SMD_Wuerth-WE-PD-Typ-LS_Handsoldering
- L2: footprint (none) -> Choke_SMD:Choke_SMD_12x12mm_h4.5mm
- Q1: footprint (none) -> toni:SO8_WITH_EP
- SMA_E1: footprint (none) -> toni:SMA_EDGE
- SW1, SW2: footprint (none) -> toni:EVQP7A
- U4: footprint (none) -> toni:Conn_03x08
- X1: footprint (none) -> toni:CRYSTAL_MT
Changed lines of the file:
@@
 EESchema Schematic File Version 2
-LIBS:SMA_EDGE
 LIBS:power
 LIBS:device
@@
 LIBS:contrib
 LIBS:valves
-LIBS:Resonator_3pins
-LIBS:rx5808
-LIBS:tps62160
-LIBS:Rafi
 LIBS:toni
-LIBS:rx5808_4button-cache
+LIBS:TX5823-cache
 EELAYER 25 0
 EELAYER END
@@
 F 0 "SW1" H 8000 5510 50  0000 C CNN
 F 1 "SW_PUSH" H 7850 5320 50  0000 C CNN
-F 2 "" H 7850 5400 60  0001 C CNN
+F 2 "toni:EVQP7A" H 7850 5400 60  0001 C CNN
 F 3 "" H 7850 5400 60  0000 C CNN
 	1    7850 5400
@@
 F 0 "X1" H 12550 6790 30  0000 C CNN
 F 1 "27MHz" H 12580 6590 30  0000 L CNN
-F 2 "" H 12550 6700 60  0001 C CNN
+F 2 "toni:CRYSTAL_MT" H 12550 6700 60  0001 C CNN
 F 3 "" H 12550 6700 60  0000 C CNN
 F 4 "NDK NX3225SA-27.000MHZ-STD-CSR-1" H 12550 6700 60  0001 C CNN "Bestellnummer"
@@
 F 0 "Q1" H 4960 2670 60  0000 R CNN
 F 1 "MOS_N" H 4960 2350 60  0000 R CNN
-F 2 "" H 4950 2500 60  0001 C CNN
+F 2 "toni:SO8_WITH_EP" H 4950 2500 60  0001 C CNN
 F 3 "" H 4950 2500 60  0000 C CNN
 F 4 " CSD18504Q5A" H 4950 2500 60  0001 C CNN "Teilenummer"
@@
 F 0 "L2" V 5300 3050 40  0000 C CNN
 F 1 "15uH" V 5450 3050 40  0000 C CNN
-F 2 "" H 5350 3050 60  0001 C CNN
+F 2 "Choke_SMD:Choke_SMD_12x12mm_h4.5mm" H 5350 3050 60  0001 C CNN
 F 3 "" H 5350 3050 60  0000 C CNN
 F 4 "MSS1210-153MEB" V 5350 3050 60  0001 C CNN "Teilenummer"
@@
 F 0 "L1" V 4750 8100 40  0000 C CNN
 F 1 "INDUCTOR" V 4900 8100 40  0000 C CNN
-F 2 "" H 4800 8100 60  0001 C CNN
+F 2 "Choke_SMD:Choke_SMD_Wuerth-WE-PD-Typ-LS_Handsoldering" H 4800 8100 60  0001 C CNN
 F 3 "" H 4800 8100 60  0000 C CNN
 	1    4800 8100
@@
 F 0 "U4" H 9850 10000 60  0000 C CNN
 F 1 "CONN_03X08" H 9200 10000 60  0000 C CNN
-F 2 "" H 9600 10450 60  0001 C CNN
+F 2 "toni:Conn_03x08" H 9600 10450 60  0001 C CNN
 F 3 "" H 9600 10450 60  0000 C CNN
 	1    9400 10300
@@
 F 0 "SW2" H 14450 9610 50  0000 C CNN
 F 1 "SW_PUSH" H 14300 9420 50  0000 C CNN
-F 2 "" H 14300 9500 60  0001 C CNN
+F 2 "toni:EVQP7A" H 14300 9500 60  0001 C CNN
 F 3 "" H 14300 9500 60  0000 C CNN
 	1    14300 9500
@@
 F 0 "SMA_E1" H 15200 1850 60  0000 C CNN
 F 1 "SMA_EDGE" H 15200 1750 60  0000 C CNN
-F 2 "" H 15050 1550 60  0000 C CNN
+F 2 "toni:SMA_EDGE" H 15050 1550 60  0001 C CNN
 F 3 "" H 15050 1550 60  0000 C CNN
 	1    15050 1550
