File: TX5823_backup_mit_12V_Buck_Boost/TX5823.sch (KiCad schematic (older format))
At the start: 73 parts, among them IC1 ATMEGA328P-A, IC2 ATTINY13A-SS, P1 Akku_in, P2 ISP, P3 Mavlink, Q3 MOSFET_N, SW1 SW_PUSH, SW2 SW_PUSH, U2 TPS54531, U3 TPS7A7200RGT, U4 CONN_03X08, U5 OPTO-TRANSISTOR4, U6 TX5823, U7 MAX7456_DS, U8 OPTO-TRANSISTOR4, X1 27MHz, Y1 16MHz

Commit message: 12V Wandler entfernt
Parts:
- added C10: Ccomp, Capacitors_SMD:C_0805, symbol C
- added C12: Cvccx, Capacitors_SMD:C_0402, symbol C
- added C13: Cvcc, Capacitors_SMD:C_0402, symbol C
- added C15: Cboot, Capacitors_SMD:C_0805, symbol C
- added C18: Cout, Capacitors_SMD:c_elec_8x10, symbol CP2
- added C38: 1uF/50V, Capacitors_SMD:C_1206, symbol C
- added C4: Css, Capacitors_SMD:C_0805, symbol C
- added C6: Cin, Capacitors_SMD:C_1206, symbol C
- added C7: Ccomp2, Capacitors_SMD:C_0805, symbol C
- added C9: Cinx, Capacitors_SMD:C_0805, symbol C
- added D2, D5: DIODESCH, Diodes_SMD:Diode-SMC_Standard, symbol DIODESCH
- added L2: 15uH, Choke_SMD:Choke_SMD_12x12mm_h4.5mm, symbol INDUCTOR
- added Q1: MOS_N, toni:SO8_WITH_EP, symbol MOS_N
- added Q2: MOS_N, symbol MOS_N
- added R1: Ruv1, Resistors_SMD:R_0402, symbol R
- added R2: Ruv2, Resistors_SMD:R_0402, symbol R
- added R3: Rt, Resistors_SMD:R_0402, symbol R
- added R4: Renable, Resistors_SMD:R_0402, symbol R
- added R5: Rcomp, Resistors_SMD:R_0402, symbol R
- added R7: Rfbb, Resistors_SMD:R_0402, symbol R
- added R8: Rfbt, Resistors_SMD:R_0402, symbol R
- added R9: Rsense, Resistors_SMD:R_1206, symbol R
- added U1: LM25118, toni:TSSOP-20_4.4x6.5mm_Pitch0.65mm_EP, symbol LM25118
- C2: value 220pF -> Cramp; footprint Capacitors_SMD:C_0402 -> Capacitors_SMD:C_0805; Teilenummer (none) -> CC0805KRX7R9BB391
- Q3: footprint toni:SOT23_GDS -> (none)
Connections:
- net +12V: now also C18.1, C38.1, D5.2 (K), R8.1, U1.10 (VOUT)
- net +3.3V: no longer C2.1
- net Akku+: now also C6.1, C9.1, Q1.D, R1.1, R4.1, U1.1 (VIN)
- net GND: now also C2.2, C12.1, C13.2, C18.2, C38.2, C4.2, C6.2, C9.2, Q2.S, R2.2, R3.2, R7.1, R9.2, U1.13 (CSG), U1.14 (PGND), U1.21 (EP), U1.6 (AGND); no longer C26.2, C27.2
- net at U3.2 (FB): now also C26.2, C27.2; no longer C2.2
- new net: D2.1 (A), R9.1, U1.12 (CS)
- new net: Q2.G, U1.15 (LO)
- new net: C13.1, U1.16 (VCC)
- new net: C12.2, U1.17 (VCCX)
- new net: C15.2, U1.18 (HB)
- new net: Q1.G, U1.19 (HO)
- new net: R1.2, R2.1, U1.2 (UVLO)
- new net: C15.1, D2.2 (K), L2.1, Q1.S, U1.20 (HS)
- new net: R3.1, U1.3 (RT)
- new net: R4.2, U1.4 (EN)
- new net: C2.1, U1.5 (RAMP)
- new net: C4.1, U1.7 (SS)
- new net: C10.2, C7.2, R7.2, R8.2, U1.8 (FB)
- new net: C10.1, R5.1, U1.9 (COMP)
- new net: D5.1 (A), L2.2, Q2.D
- new net: C7.1, R5.2
- no-connect marks 27 -> 28
Other:
- note added: "12V Buck Boost\nVinMin 8V\nVinMax=30V\nVout=12V\nIout= 2A"
- note added: "TODO:\nSMA Buchse\nEingangsfilterung (spule und diode)"
- note removed: "TODO:\nEingangsfilterung (spule und diode)\n12V Aufsteckplatine"
- moved on the sheet: C26, C27
